Commit message: update eva urdf

File: urdf/eva_description/urdf/eva_description.urdf (robot description, URDF)
Before this commit: robot eva_description, 10 links, 9 joints
Links:
- link gripper_1: geometry collision mesh filename=../meshes/gripper_1.dae; visual mesh filename=../meshes/gripper_1.dae
- link gripper_2: geometry collision mesh filename=../meshes/gripper_2.dae; visual mesh filename=../meshes/gripper_2.dae
- link model_0: geometry collision mesh filename=../meshes/model_0.dae; visual mesh filename=../meshes/model_0.dae
- link model_1: geometry collision mesh filename=../meshes/model_1.dae; visual mesh filename=../meshes/model_1.dae
- link model_2: geometry collision mesh filename=../meshes/model_2.dae; visual mesh filename=../meshes/model_2.dae
- link model_3: geometry collision mesh filename=../meshes/model_3.dae; visual mesh filename=../meshes/model_3.dae
- link model_4: geometry collision mesh filename=../meshes/model_4.dae; visual mesh filename=../meshes/model_4.dae
- link model_5: geometry collision mesh filename=../meshes/model_5.dae; visual mesh filename=../meshes/model_5.dae
- link model_6: geometry collision mesh filename=../meshes/model_6.dae; visual mesh filename=../meshes/model_6.dae
