Commit message: update URDF UR5e

File: frontend/public/urdf/ur5_description/urdf/ur5_robot.urdf (robot description, URDF)
Before this commit: robot ur5, 11 links, 10 joints
Links:
- removed link tool0
- added link tool_point, mass 0
Joints:
- joint wrist_3_link-tool0_fixed_joint: child tool0 -> tool_point

Commit message: updated UR5e

File: frontend/public/urdf/ur5_description/urdf/ur5_robot.urdf (robot description, URDF)
Before this commit: robot ur5, 11 links, 10 joints
Joints:
- joint world_joint: origin xyz=0.0 0.0 0.0 rpy=0.0 0.0 0.0 -> xyz=0.0 0.0 0.07863 rpy=0.0 0.0 0.0

Commit message: updated UR5e URDF

File: frontend/public/urdf/ur5_description/urdf/ur5_robot.urdf (robot description, URDF)
Before this commit: robot ur5, 11 links, 10 joints
Links:
- removed link ee_link
- added link base_link_inertia, mass 4.0; collision mesh filename=../meshes/collision/base.stl; visual mesh filename=../meshes/visual/base.dae
- added link flange
- added link ft_frame
- link base: mass 0 -> None
- link base_link: mass 4.0 -> None; geometry 
- link forearm_link: mass 2.275 -> 2.846
- link shoulder_link: mass 3.7 -> 3.761
- link tool_point: mass 0 -> None
- link upper_arm_link: mass 8.393 -> 8.058
- link wrist_1_link: mass 1.219 -> 1.37
- link wrist_2_link: mass 1.219 -> 1.3
- link wrist_3_link: mass 0.1879 -> 0.365
Joints:
- removed joint ee_fixed_joint
- removed joint world_joint
- removed joint wrist_3_link-tool0_fixed_joint
- added joint base_joint: type fixed, parent world, child base_link, origin xyz=0 0 0 rpy=0 0 0
- added joint base_link-base_link_inertia: type fixed, parent base_link, child base_link_inertia, origin xyz=0 0 0 rpy=0 0 3.141592653589793
- added joint flange-tool_point: type fixed, parent flange, child tool_point, origin xyz=0 0 0 rpy=1.5707963267948966 0 1.5707963267948966
- added joint wrist_3-flange: type fixed, parent wrist_3_link, child flange, origin xyz=0 0 0 rpy=0 -1.5707963267948966 -1.5707963267948966
- added joint wrist_3_link-ft_frame: type fixed, parent wrist_3_link, child ft_frame, origin xyz=0 0 0 rpy=3.141592653589793 0 0
- joint base_link-base_fixed_joint: origin xyz=0 0 0 rpy=0 0 -3.14159265359 -> xyz=0 0 0 rpy=0 0 3.141592653589793
- joint elbow_joint: axis 0 1 0 -> 0 0 1; limit lower=-3.14159265359 upper=3.14159265359 effort=150.0 velocity=3.15 -> lower=-3.141592653589793 upper=3.141592653589793 effort=150.0 velocity=3.141592653589793; origin xyz=0.0 -0.1197 0.425 rpy=0.0 0.0 0.0 -> xyz=-0.425 0 0 rpy=0 0 0
- joint shoulder_lift_joint: axis 0 1 0 -> 0 0 1; limit lower=-6.28318530718 upper=6.28318530718 effort=150.0 velocity=3.15 -> lower=-6.283185307179586 upper=6.283185307179586 effort=150.0 velocity=3.141592653589793; origin xyz=0.0 0.13585 0.0 rpy=0.0 1.57079632679 0.0 -> xyz=0 0 0 rpy=1.570796327 0 0
- joint shoulder_pan_joint: limit lower=-6.28318530718 upper=6.28318530718 effort=150.0 velocity=3.15 -> lower=-6.283185307179586 upper=6.283185307179586 effort=150.0 velocity=3.141592653589793; origin xyz=0.0 0.0 0.089159 rpy=0.0 0.0 0.0 -> xyz=0 0 0.1625 rpy=0 0 0; parent base_link -> base_link_inertia
- joint wrist_1_joint: axis 0 1 0 -> 0 0 1; limit lower=-6.28318530718 upper=6.28318530718 effort=28.0 velocity=3.2 -> lower=-6.283185307179586 upper=6.283185307179586 effort=28.0 velocity=3.141592653589793; origin xyz=0.0 0.0 0.39225 rpy=0.0 1.57079632679 0.0 -> xyz=-0.3922 0 0.1333 rpy=0 0 0
- joint wrist_2_joint: limit lower=-6.28318530718 upper=6.28318530718 effort=28.0 velocity=3.2 -> lower=-6.283185307179586 upper=6.283185307179586 effort=28.0 velocity=3.141592653589793; origin xyz=0.0 0.093 0.0 rpy=0.0 0.0 0.0 -> xyz=0 -0.0997 -2.044881182297852e-11 rpy=1.570796327 0 0
- joint wrist_3_joint: axis 0 1 0 -> 0 0 1; limit lower=-6.28318530718 upper=6.28318530718 effort=28.0 velocity=3.2 -> lower=-6.283185307179586 upper=6.283185307179586 effort=28.0 velocity=3.141592653589793; origin xyz=0.0 0.0 0.09465 rpy=0.0 0.0 0.0 -> xyz=0 0.0996 -2.042830148012698e-11 rpy=1.570796326589793 3.141592653589793 3.141592653589793
